File: SHEET10.kicad_sch (KiCad schematic)
At the start: 42 parts, among them J1 I/O_CONNECTOR, J2 I/O_CONNECTOR, J3 I/O_CONNECTOR, J4 I/O_CONNECTOR, J5 I/O_CONNECTOR, P1 POWER_CON, P2 POWER_CON

Commit message: 3d view
Other:
- note added: "KevJu: Use 10uF 25V tantalum caps. The footprint is set up for 3-lead or 2-lead with 2.5mm spacing. Center terminal is most posistive. Do not use 5.0mm lead space caps."
- note added: "KevJu: Use 47nF or 100nF 50V ceramic caps with 2.5mm or 5.0mm lead spacing. No polarity."
- note removed: "Kev-Ju: Use 10uF 25V tantalum caps. The footprint is set up for 3-lead or 2-lead with 2.5mm spacing. Center terminal is most posistive. Do not use 5.0mm lead space caps."
- note removed: "Kev-Ju: Use 47nF or 100nF 50V ceramic caps with 2.5mm or 5.0mm lead spacing. No polarity."
Changed lines of the file:
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@@
 		)
 	)
-	(text "Kev-Ju:\nUse 47nF or 100nF 50V ceramic caps \nwith 2.5mm or 5.0mm lead spacing.\nNo polarity."
+	(text "KevJu:\nUse 47nF or 100nF 50V ceramic caps \nwith 2.5mm or 5.0mm lead spacing.\nNo polarity."
 		(exclude_from_sim no)
 		(at 161.29 198.12 0)
@@
 		)
 	)
-	(text "Kev-Ju:\nUse 10uF 25V tantalum caps. \nThe footprint is set up for 3-lead \nor 2-lead with 2.5mm spacing. \nCenter terminal is most posistive.\n\nDo not use 5.0mm lead space caps."
+	(text "KevJu:\nUse 10uF 25V tantalum caps. \nThe footprint is set up for 3-lead \nor 2-lead with 2.5mm spacing. \nCenter terminal is most posistive.\n\nDo not use 5.0mm lead space caps."
 		(exclude_from_sim no)
 		(at 245.11 260.35 0)
@@
 		)
 		(stroke
-			(width 0)
+			(width 0.254)
 			(type default)
 			(color 194 194 194 1)
@@
 		)
 		(stroke
-			(width 0)
-			(type solid)
+			(width 0.254)
+			(type default)
 			(color 194 194 194 1)
 		)
@@
 		)
 		(stroke
-			(width 0)
+			(width 0.254)
 			(type default)
 			(color 194 194 194 1)
@@
 		)
 		(stroke
-			(width 0)
+			(width 0.254)
 			(type default)
 			(color 194 194 194 1)
@@
 		)
 		(stroke
-			(width 0)
+			(width 0.254)
 			(type default)
 			(color 194 194 194 1)
@@
 		)
 		(stroke
-			(width 0)
+			(width 0.254)
 			(type default)
 			(color 194 194 194 1)
@@
 		)
 		(stroke
-			(width 0)
-			(type solid)
+			(width 0.254)
+			(type default)
 			(color 194 194 194 1)
 		)
@@
 		)
 		(stroke
-			(width 0)
-			(type solid)
+			(width 0.254)
+			(type default)
 			(color 194 194 194 1)
 		)
@@
 		)
 		(stroke
-			(width 0)
+			(width 0.254)
 			(type default)
 			(color 194 194 194 1)
@@
 		)
 		(stroke
-			(width 0)
-			(type solid)
+			(width 0.254)
+			(type default)
 			(color 194 194 194 1)
 		)
@@
 		)
 		(stroke
-			(width 0)
-			(type solid)
+			(width 0.254)
+			(type default)
 			(color 194 194 194 1)
 		)
@@
 		)
 		(stroke
-			(width 0)
+			(width 0.254)
 			(type default)
 			(color 194 194 194 1)
@@
 		)
 		(stroke
-			(width 0)
+			(width 0.254)
 			(type default)
 			(color 194 194 194 1)
@@
 		)
 		(stroke
-			(width 0)
+			(width 0.254)
 			(type default)
 			(color 194 194 194 1)
@@
 		)
 		(stroke
-			(width 0)
+			(width 0.254)
 			(type default)
 			(color 194 194 194 1)
@@
 		)
 		(stroke
-			(width 0)
+			(width 0.254)
 			(type default)
 			(color 194 194 194 1)
@@
 		)
 		(stroke
-			(width 0)
-			(type solid)
+			(width 0.254)
+			(type default)
 			(color 194 194 194 1)
 		)
@@
 		)
 		(stroke
-			(width 0)
-			(type solid)
+			(width 0.254)
+			(type default)
 			(color 194 194 194 1)
 		)
@@
 		)
 		(stroke
-			(width 0)
+			(width 0.254)
 			(type default)
 			(color 194 194 194 1)
@@
 		)
 		(stroke
-			(width 0)
+			(width 0.254)
 			(type default)
 			(color 194 194 194 1)
@@
 		)
 		(stroke
-			(width 0)
+			(width 0.254)
 			(type default)
 			(color 194 194 194 1)

Commit message: added BOM
Parts:
- C12, C13, C14, C17, C2, C23, C25, C3, C38, C40, C42, C44, C6: Link (none) -> https://www.digikey.com/en/products/detail/kyocera-avx/TAP1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
- C18, C19, C20, C21, C22, C24, C26, C27, C28, C29, C30, C31, C32, C33, C34, C35, C36, C37, C39, C41, C43, C45: Link (none) -> https://www.digikey.com/en/products/detail/vishay-beyschlag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; Note (none) -> No reason not to use 100n here
- J1, J2, J3, J4, J5: Link (none) -> https://www.digikey.com/en/products/detail/edac-inc/395-062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
- P1, P2: Link (none) -> https://www.digikey.com/en/products/detail/molex/0366420001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; Note (none) -> It's black instead of white, but it's the right shape.
