File: SHEET2.kicad_sch (KiCad schematic)
At the start: 20 parts, among them J8 +RUN, U5 74LS30, U50 74LS02, U51 74LS04, U52 74LS00, U64 74LS20, U67 74LS74, U81 74LS00, U82 74LS74, U83 74LS04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

Commit message: Fixed LS and S parts
Parts:
- U81: value 74LS00 -> 74S00
- U82: value 74LS74 -> 74S74
- U84: value 74LS10 -> 74S10
- U97: value 74LS08 -> 74S08
Changed lines of the file:
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@@
 			)
 		)
-		(property "Value" "74LS10"
+		(property "Value" "74S10"
 			(at 127 73.66 0)
 			(effects
@@
 			)
 		)
-		(property "Value" "74LS74"
+		(property "Value" "74S74"
 			(at 227.33 59.563 0)
 			(effects
@@
 			)
 		)
-		(property "Value" "74LS08"
+		(property "Value" "74S08"
 			(at 322.58 91.44 0)
 			(effects
@@
 			)
 		)
-		(property "Value" "74LS08"
+		(property "Value" "74S08"
 			(at 257.81 119.38 0)
 			(effects
@@
 			)
 		)
-		(property "Value" "74LS08"
+		(property "Value" "74S08"
 			(at 289.56 191.77 0)
 			(effects
@@
 			)
 		)
-		(property "Value" "74LS10"
+		(property "Value" "74S10"
 			(at 129.54 189.23 0)
 			(effects
@@
 			)
 		)
-		(property "Value" "74LS00"
+		(property "Value" "74S00"
 			(at 87.63 181.61 0)
 			(effects

Commit message: added BOM
Parts:
- J8: value +RUN -> RUN; now not fitted
- JP1: value Jumper_2_Open -> 1x2; now not fitted
- R11: Link (none) -> https://www.digikey.com/en/products/detail/yageo/MFR-25FTE5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
- R12: Link (none) -> https://www.digikey.com/en/products/detail/yageo/MFR-25FRF5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
- RN1: Link (none) -> https://www.digikey.com/en/products/detail/bourns-inc/4116R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
- TD2: Link (none) -> https://www.digikey.com/en/products/detail/yageo/MFR-25FTE5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; Note (none) -> Use a 470 Ohm resistor here
- U5, U50, U51, U52, U64, U67, U81, U82, U83, U96, U97, U98, U99: Link (none) -> https://www.digikey.com/en/products/detail/texas-instrument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
- U84: Link (none) -> https://www.mouser.com/ProductDetail/Texas-Instruments/SN74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
