File: SHEET5.kicad_sch (KiCad schematic)
At the start: 13 parts, among them U13 74LS245, U14 74LS245, U15 74LS244, U16 74LS244, U27 74LS02, U28 8K_X_8ROS, U29 8K_X_8ROS, U30 8K_X_8ROS, U31 8K_X_8ROS, U32 8K_X_8ROS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

Commit message: added BOM
Parts:
- R20: Link (none) -> https://www.digikey.com/en/products/detail/yageo/MFR-25FTE5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
- RN1: Link (none) -> https://www.digikey.com/en/products/detail/bourns-inc/4116R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
- U13, U14, U15, U16, U27: Link (none) -> https://www.digikey.com/en/products/detail/texas-instrument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
- U28, U29, U30, U31, U32, U33: Link (none) -> https://www.minuszerodegrees.net/5150/motherboard/IBM%20515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
Other:
- moved on the sheet: R20, RN1B, RN1C, RN1F, RN1G, U13, U14, U15, U16, U27A, U27B, U27D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
