File: SHEET9.kicad_sch (KiCad schematic)
At the start: 18 parts, among them J7 KBD, SW1 DIP_SW8, SW2 DIP_SW8, U23 74LS244, U24 74LS322, U26 74LS175, U36 8255A-5, U63 74LS38, U80 74LS125, U82 74LS74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

Commit message: Fixed LS and S parts
Parts:
- U82: value 74LS74 -> 74S74
Changed lines of the file:
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@@
 			)
 		)
-		(property "Value" "74LS74"
+		(property "Value" "74S74"
 			(at 337.82 171.323 0)
 			(effects

Commit message: added BOM
Parts:
- C10: Link (none) -> https://www.digikey.com/en/products/detail/vishay-beyschlag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; Note (none) -> No reason not to use 100n here
- C11, C15, C7: Link (none) -> https://www.digikey.com/en/products/detail/vishay-beyschlag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
- J7: Link (none) -> https://www.digikey.com/en/products/detail/kycon-inc/KCDX-5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
- RN1, RN3: Link (none) -> https://www.digikey.com/en/products/detail/bourns-inc/4116R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
- RN2: Link (none) -> https://www.digikey.com/en/products/detail/bourns-inc/4116R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; Note (none) -> There is no reason to use 8.2k here, another 4.7k will work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
- SW1, SW2: Link (none) -> https://www.digikey.com/en/products/detail/te-connectivity-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
- U23, U26, U63, U80, U82, U99: Link (none) -> https://www.digikey.com/en/products/detail/texas-instrument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
- U24: Link (none) -> https://www.jameco.com/z/AM25LS22PC-Advanced-Micro-Devices-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; Note (none) -> *** Investigate replacing this
- U36: Link (none) -> https://www.jameco.com/z/P8255A-5-Intel-Corporation-IC-8255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
