File: SHEET3.kicad_sch (KiCad schematic)
At the start: 11 parts, among them U46 74LS138, U47 74LS138, U48 74LS138, U49 74LS08, U50 74LS02, U51 74LS04, U64 74LS20, U65 74LS138, U66 74LS138, U81 74LS00

Commit message: Fixed LS and S parts
Parts:
- U49: value 74LS08 -> 74S08
- U65: value 74LS138 -> 74S138
- U81: value 74LS00 -> 74S00
Changed lines of the file:
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@@
 			)
 		)
-		(property "Value" "74LS138"
+		(property "Value" "74S138"
 			(at 176.53 204.4446 0)
 			(effects
@@
 			)
 		)
-		(property "Value" "74LS00"
+		(property "Value" "74S00"
 			(at 177.8 255.27 0)
 			(effects
@@
 			)
 		)
-		(property "Value" "74LS00"
+		(property "Value" "74S00"
 			(at 175.26 100.33 0)
 			(effects
@@
 			)
 		)
-		(property "Value" "74LS08"
+		(property "Value" "74S08"
 			(at 246.38 204.47 0)
 			(effects
@@
 			)
 		)
-		(property "Value" "74LS08"
+		(property "Value" "74S08"
 			(at 246.38 218.44 0)
 			(effects
@@
 			)
 		)
-		(property "Value" "74LS08"
+		(property "Value" "74S08"
 			(at 246.38 190.5 0)
 			(effects
@@
 			)
 		)
-		(property "Value" "74LS08"
+		(property "Value" "74S08"
 			(at 246.38 176.53 0)
 			(effects
@@
 			)
 		)
-		(property "Value" "74LS00"
+		(property "Value" "74S00"
 			(at 288.29 129.54 0)
 			(effects

Commit message: added BOM
Parts:
- TD1: Note (none) -> Ebay, or possibly use DS1100Z-100+ with an adapter PCB
- U46, U47, U48, U49, U50, U51, U64, U65, U66, U81: Link (none) -> https://www.digikey.com/en/products/detail/texas-instrument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

Commit message: fixed td1 bom
Parts:
- TD1: Link (none) -> https://www.questcomp.com/part/4/ds1000m-125/177328069; Note Ebay, or possibly use DS1100Z-100+ with an adapter PCB -> https://www.questcomp.com/part/4/ds1000m-100/177328066 prob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
Changed lines of the file:
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@@
 			)
 		)
-		(property "Link" ""
+		(property "Link" "https://www.questcomp.com/part/4/ds1000m-125/177328069"
 			(at 213.36 110.49 0)
 			(effects
@@
 			)
 		)
-		(property "Note" "Ebay, or possibly use DS1100Z-100+ with an adapter PCB"
+		(property "Note" "https://www.questcomp.com/part/4/ds1000m-100/177328066 probably also works"
 			(at 213.36 110.49 0)
 			(effects
